File: baseline/02-two-layer/02-two-layer.kicad_pcb (KiCad board)
At the start: 2 copper layers, 52.1 x 46.4 mm, 15 parts, among them P1 IN, P2 OUT, P3 POWER, P4 CONN_2, P5 MOUNTING_HOLE, P6 MOUNTING_HOLE, P7 MOUNTING_HOLE, P8 MOUNTING_HOLE, U1 ECC83

Commit message: feat(bundle): route nets as a seated bundle rather than one after another
Sequential routing has a failure no ordering can fix. A gap wide enough
for two tracks: the first net through it is asked, alone, where a rubber
band would sit, and a rubber band sits in the middle. The second finds
the gap full. Re-routing the first puts it back exactly where it was --
the taut path is deterministic -- so ripping up and re-ordering only
swaps who is stranded.

Routing now happens in two stages. Every connection is first routed
against the static obstacles alone, which says which gap it *wants* --
including connections that a sequential pass would have blocked, so a
stranded net still gets a say. Gaps are then counted,
floor((D - c) / (w + c)) tracks each, contending nets are ordered across
each gap and given slots, and every connection is routed again against
obstacles inflated by its own slot's share. Nothing is pushed: each net
is simply handed a problem that already contains the others.

The slack in a gap has to be divided rather than handed to every net.
Giving each the full band let them all drift to the inside of it and end
up 1.5 apart where 2.0 was required; folding an equal share into the
stride fixes it, and any position in one band is then a full pitch from
any position in the next.

Slot assignment is a model, so the arrangement is verified afterwards on
real geometry and anything still too close is routed the old way. That
settling pass also reconsiders which layer a connection sits on --
choosing it before the contention is known left a two-layer board using
one layer and stranding a net on it.

Results are unchanged on all three boards, and that is the honest
finding rather than a disappointment to hide:

  ecc83-pp F.Cu        19/20 -> 19/20
  ecc83-pp F.Cu+B.Cu   20/20 -> 20/20
  sonde xilinx         63/66 -> 63/66, 0 DRC either way

The mechanism is proven on the case it exists for -- tests/test_bundle.py
shows the second net raising NoPathFound sequentiall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
Routing:
- net Net-(U1A-G): track 48.7 -> 19.5 mm
- net Net-(P1-PM): track 47.8 -> 27.6 mm
- net Net-(U1B-K): track 28.3 -> 16.1 mm
- net Net-(P3-P1): track 33.6 -> 23.5 mm
- net GND: track 78.2 -> 85.3 mm
Changed lines of the file:
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@@
 	(segment
 		(start 141.605 94.695)
-		(end 139.046033 96.591777)
-		(width 0.8)
-		(layer "F.Cu")
-		(net 1)
-	)
-	(segment
-		(start 139.046033 96.591777)
-		(end 138.913032 96.697209)
-		(width 0.8)
-		(layer "F.Cu")
-		(net 1)
-	)
-	(segment
-		(start 138.913032 96.697209)
 		(end 128.27 105.711)
 		(width 0.8)
@@
 	(segment
 		(start 164.465 117.475)
-		(end 162.86901 124.744612)
+		(end 164.036689 106.943892)
 		(width 0.8)
-		(layer "F.Cu")
+		(layer "B.Cu")
+		(net 5)
+	)
+	(segment
+		(start 164.036689 106.943892)
+		(end 164.036 106.91)
+		(width 0.8)
+		(layer "B.Cu")
+		(net 5)
+	)
+	(segment
+		(start 164.036 106.91)
+		(end 164.036 103.91)
+		(width 0.8)
+		(layer "B.Cu")
 		(net 5)
 	)
 	(arc
-		(start 162.86901 124.744612)
-		(mid 164.156812 126.699673)
-		(end 166.077241 125.360774)
+		(start 164.036 103.91)
+		(mid 164.076482 103.653318)
+		(end 164.193999 103.421555)
 		(width 0.8)
-		(layer "F.Cu")
+		(layer "B.Cu")
 		(net 5)
 	)
 	(segment
-		(start 166.077241 125.360774)
-		(end 167.286071 118.02775)
-		(width 0.8)
-		(layer "F.Cu")
-		(net 5)
-	)
-	(segment
-		(start 167.286071 118.02775)
-		(end 167.292505 117.983805)
-		(width 0.8)
-		(layer "F.Cu")
-		(net 5)
-	)
-	(segment
-		(start 167.292505 117.983805)
-		(end 168.697243 107.015951)
-		(width 0.8)
-		(layer "F.Cu")
-		(net 5)
-	)
-	(segment
-		(start 168.697243 107.015951)
-		(end 168.704 106.91)
-		(width 0.8)
-		(layer "F.Cu")
-		(net 5)
-	)
-	(segment
-		(start 168.704 106.91)
-		(end 168.704 103.91)
-		(width 0.8)
-		(layer "F.Cu")
-		(net 5)
-	)
-	(arc
-		(start 168.704 103.91)
-		(mid 168.663518 103.653318)
-		(end 168.546001 103.421555)
-		(width 0.8)
-		(layer "F.Cu")
-		(net 5)
-	)
-	(segment
-		(start 168.546001 103.421555)
+		(start 164.193999 103.421555)
 		(end 166.37 100.41)
 		(width 0.8)
-		(layer "F.Cu")
+		(layer "B.Cu")
 		(net 5)
 	)
 	(segment
 		(start 156.21 95.885)
-		(end 148.940388 94.28901)
-		(width 0.8)
-		(layer "F.Cu")
-		(net 13)
-	)
-	(arc
-		(start 148.940388 94.28901)
-		(mid 147.253886 94.944385)
-		(end 147.205679 96.753108)
-		(width 0.8)
-		(layer "F.Cu")
-		(net 13)
-	)
-	(segment
-		(start 147.205679 96.753108)
-		(end 154.241468 107.972667)
-		(width 0.8)
-		(layer "F.Cu")
-		(net 13)
-	)
-	(arc
-		(start 154.241468 107.972667)
-		(mid 154.424415 108.356379)
-		(end 154.514895 108.771733)
-		(width 0.8)
-		(layer "F.Cu")
-		(net 13)
-	)
-	(segment
-		(start 154.514895 108.771733)
 		(end 154.825 111.885)
 		(width 0.8)
-		(layer "F.Cu")
+		(layer "B.Cu")
 		(net 13)
 	)
@@
 	(segment
 		(start 141.605 99.695)
-		(end 143.31117 95.367711)
-		(width 0.8)
-		(layer "F.Cu")
-		(net 2)
-	)
-	(arc
-		(start 143.31117 95.367711)
-		(mid 142.784293 93.290428)
-		(end 140.647172 93.130992)
-		(width 0.8)
-		(layer "F.Cu")
-		(net 2)
-	)
-	(segment
-		(start 140.647172 93.130992)
 		(end 128.27 100.711)
 		(width 0.8)
-		(layer "F.Cu")
+		(layer "B.Cu")
 		(net 2)
 	)
@@
 	(segment
 		(start 143.615 111.885)
-		(end 147.305307 117.442134)
-		(width 0.8)
-		(layer "F.Cu")
-		(net 12)
-	)
-	(arc
-		(start 147.305307 117.442134)
-		(mid 147.522308 117.88996)
-		(end 147.612019 118.379439)
-		(width 0.8)
-		(layer "F.Cu")
-		(net 12)
-	)
-	(segment
-		(start 147.612019 118.379439)
-		(end 148.2105 131.299003)
-		(width 0.8)
-		(layer "F.Cu")
-		(net 12)
-	)
-	(arc
-		(start 148.2105 131.299003)
-		(mid 148.753309 132.69038)
-		(end 150.02852 133.467817)
-		(width 0.8)
-		(layer "F.Cu")
-		(net 12)
-	)
-	(arc
-		(start 150.02852 133.467817)
-		(mid 152.013952 133.002329)
-		(end 152.875708 131.154087)
-		(width 0.8)
-		(layer "F.Cu")
-		(net 12)
-	)
-	(segment
-		(start 152.875708 131.154087)
 		(end 152.675 118.465)
 		(width 0.8)
-		(layer "F.Cu")
+		(layer "B.Cu")
 		(net 12)
 	)
@@
 	)
 	(segment
+		(start 141.605 94.695)
+		(end 148.59 95.885)
+		(width 0.8)
+		(layer "F.Cu")
+		(net 1)
+	)
+	(segment
