File: results/_work/ecc83-pp-relaxed.kicad_pcb (KiCad board)
At the start: 2 copper layers, 52.1 x 46.4 mm, 15 parts, among them P1 IN, P2 OUT, P3 POWER, P4 CONN_2, P5 MOUNTING_HOLE, P6 MOUNTING_HOLE, P7 MOUNTING_HOLE, P8 MOUNTING_HOLE, U1 ECC83

Commit message: feat(relax): settle every band at once instead of counting gaps
Replaces the portal/capacity/slot machinery with the direct thing it was
approximating. A board's copper is one arrangement, not a sequence of
decisions, so every band is re-solved against the *previous* positions of
all the others and all of them move together. Two bands contending for
the same space now both give way, which no ordering or rip-up can
produce.

The portals were scaffolding built to fake simultaneity, and they only
ever covered contention inside a narrow gap between two static obstacles.
Measurement showed why that was not enough: contention costs 30.4% of
ideal length on ecc83-pp and the slot model recovered none of it, because
the bands that detour are detouring around other *bands*, in open copper,
where no such gap exists.

Which layer a band sits on is settled in the same loop. Fixing it
beforehand -- each connection taking whichever layer was shortest for it
alone -- puts every band on one face, which the relaxation is then good
enough to make work while being materially longer than spreading out.

An earlier version also annealed the band-to-band clearance from soft to
solid, arguing that the taut solver treats other copper as walls and
walls do not yield. The argument is sound and the effect is nil: the
finished route on ecc83-pp is identical at 0.30, 0.60 and 1.00 hardness.
Bands have room to go around each other far more often than they need to
pass through, so the softening is gone rather than kept on a plausible
story.

Sequential settling versus joint relaxation, same boards, same process:

  ecc83-pp F.Cu        19/20  305.3mm  ->  20/20  292.9mm
  ecc83-pp F.Cu+B.Cu   20/20  239.5mm  ->  20/20  239.5mm
  sonde xilinx         63/66  690.3mm  ->  64/66  678.4mm

Where there is headroom it wins on both counts -- more connections
finished and less copper -- which is the tell that it is doing the right
thing rather than merely doing something. Zero DRC errors throughout.

Relax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
Routing:
- net Net-(U1A-G): track 48.7 -> 19.5 mm
- net GND: track 99.3 -> 85.3 mm
- net Net-(P2-P1): track 26.4 -> 16.8 mm
Changed lines of the file:
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@@
 		(end 150.826459 118.423814)
 		(width 0.8)
-		(layer "F.Cu")
+		(layer "B.Cu")
 		(net 7)
 	)
@@
 		(end 150.861284 118.105505)
 		(width 0.8)
-		(layer "F.Cu")
+		(layer "B.Cu")
 		(net 7)
 	)
@@
 		(end 152.675 108.955)
 		(width 0.8)
-		(layer "F.Cu")
+		(layer "B.Cu")
 		(net 7)
 	)
 	(segment
 		(start 148.59 95.885)
-		(end 155.859612 94.28901)
-		(width 0.8)
-		(layer "F.Cu")
-		(net 1)
-	)
-	(arc
-		(start 155.859612 94.28901)
-		(mid 156.324211 94.254996)
-		(end 156.779527 94.353466)
-		(width 0.8)
-		(layer "F.Cu")
-		(net 1)
-	)
-	(segment
-		(start 156.779527 94.353466)
-		(end 167.18351 98.222363)
-		(width 0.8)
-		(layer "F.Cu")
-		(net 1)
-	)
-	(arc
-		(start 167.18351 98.222363)
-		(mid 168.550617 99.577854)
-		(end 168.434103 101.499511)
-		(width 0.8)
-		(layer "F.Cu")
-		(net 1)
-	)
-	(segment
-		(start 168.434103 101.499511)
 		(end 166.37 105.41)
 		(width 0.8)
-		(layer "F.Cu")
+		(layer "B.Cu")
 		(net 1)
 	)
@@
 	(segment
 		(start 141.605 94.695)
-		(end 126.570383 98.401241)
-		(width 0.8)
-		(layer "F.Cu")
-		(net 1)
-	)
-	(arc
-		(start 126.570383 98.401241)
-		(mid 126.11348 98.696668)
-		(end 125.936 99.211)
-		(width 0.8)
-		(layer "F.Cu")
-		(net 1)
-	)
-	(segment
-		(start 125.936 99.211)
-		(end 125.936 102.211)
-		(width 0.8)
-		(layer "F.Cu")
-		(net 1)
-	)
-	(arc
-		(start 125.936 102.211)
-		(mid 125.976482 102.467682)
-		(end 126.093999 102.699445)
-		(width 0.8)
-		(layer "F.Cu")
-		(net 1)
-	)
-	(segment
-		(start 126.093999 102.699445)
 		(end 128.27 105.711)
 		(width 0.8)
-		(layer "F.Cu")
+		(layer "B.Cu")
 		(net 1)
 	)
@@
 	(segment
 		(start 133.985 125.095)
-		(end 126.715388 126.69099)
+		(end 130.411602 116.848046)
 		(width 0.8)
-		(layer "F.Cu")
-		(net 3)
-	)
-	(arc
-		(start 126.715388 126.69099)
-		(mid 125.241303 126.281281)
-		(end 124.752379 124.831543)
-		(width 0.8)
-		(layer "F.Cu")
+		(layer "B.Cu")
 		(net 3)
 	)
 	(segment
-		(start 124.752379 124.831543)
-		(end 125.966538 117.399679)
+		(start 130.411602 116.848046)
+		(end 130.334103 116.686489)
 		(width 0.8)
-		(layer "F.Cu")
-		(net 3)
-	)
-	(arc
-		(start 125.966538 117.399679)
-		(mid 126.057294 117.033377)
-		(end 126.205897 116.686489)
-		(width 0.8)
-		(layer "F.Cu")
+		(layer "B.Cu")
 		(net 3)
 	)
 	(segment
-		(start 126.205897 116.686489)
+		(start 130.334103 116.686489)
 		(end 128.27 112.776)
 		(width 0.8)
-		(layer "F.Cu")
+		(layer "B.Cu")
 		(net 3)
 	)
@@
 	(segment
 		(start 128.27 105.711)
-		(end 130.535378 110.944711)
+		(end 126.004622 110.944711)
 		(width 0.8)
 		(layer "F.Cu")
@@
 	)
 	(arc
-		(start 130.535378 110.944711)
-		(mid 130.586664 111.106839)
-		(end 130.604 111.276)
+		(start 126.004622 110.944711)
+		(mid 125.953336 111.106839)
+		(end 125.936 111.276)
 		(width 0.8)
 		(layer "F.Cu")
@@
 	)
 	(segment
-		(start 130.604 111.276)
-		(end 130.604 114.276)
+		(start 125.936 111.276)
+		(end 125.936 114.276)
 		(width 0.8)
 		(layer "F.Cu")
@@
 	)
 	(arc
-		(start 130.604 114.276)
-		(mid 130.563518 114.532682)
-		(end 130.446001 114.764445)
+		(start 125.936 114.276)
+		(mid 125.976482 114.532682)
+		(end 126.093999 114.764445)
 		(width 0.8)
 		(layer "F.Cu")
@@
 	)
 	(segment
-		(start 130.446001 114.764445)
+		(start 126.093999 114.764445)
 		(end 128.27 117.776)
 		(width 0.8)
@@
 	(segment
 		(start 143.615 111.885)
-		(end 147.305307 117.442134)
-		(width 0.8)
-		(layer "F.Cu")
-		(net 12)
-	)
-	(arc
-		(start 147.305307 117.442134)
-		(mid 147.522308 117.88996)
-		(end 147.612019 118.379439)
-		(width 0.8)
-		(layer "F.Cu")
-		(net 12)
-	)
-	(segment
-		(start 147.612019 118.379439)
-		(end 148.2105 131.299003)
-		(width 0.8)
-		(layer "F.Cu")
-		(net 12)
-	)
-	(arc
-		(start 148.2105 131.299003)
-		(mid 148.753309 132.69038)
-		(end 150.02852 133.467817)
-		(width 0.8)
-		(layer "F.Cu")
-		(net 12)
-	)
-	(arc
-		(start 150.02852 133.467817)
-		(mid 152.013952 133.002329)
-		(end 152.875708 131.154087)
-		(width 0.8)
-		(layer "F.Cu")
-		(net 12)
-	)
-	(segment
-		(start 152.875708 131.154087)
 		(end 152.675 118.465)
 		(width 0.8)
